Commit message: completing the xacro file and some changes on visualizer

File: urdf/field.xacro (robot description, xacro)
@@ -42,4 +42,10 @@
       <material name="white"/>
     </visual>
+    <collision>
+      <geometry>
+        <cylinder length="${scale * 0.001}" radius ="${scale * 0.75}"/>
+      </geometry>
+      <origin xyz="0 0 ${scale * 0.005}"/>
+    </collision>
   </link>
   <joint name="base_with_kickoff_line" type="fixed">
@@ -55,4 +61,10 @@
       <material name="white"/>
     </visual>
+    <collision>
+      <geometry>
+        <cylinder length="${scale * 0.001}" radius ="${scale * 0.075}"/>
+      </geometry>
+      <origin xyz="0 0 ${scale * 0.009}"/>
+    </collision>
   </link>
   <joint name="base_with_kickoff_spot" type="fixed">
@@ -68,4 +80,10 @@
       <material name="green"/>
     </visual>
+    <collision>
+      <geometry>
+        <cylinder length="${scale * 0.001}" radius ="${scale * 0.67}"/>
+      </geometry>
+      <origin xyz ="0 0 ${scale * 0.007}"/>
+    </collision>
   </link>
   <joint name="base_with_kickoff_area" type="fixed">
@@ -81,4 +99,10 @@
       <material name="white"/>
     </visual>
+    <collision>
+      <geometry>
+        <box size="${scale * 0.08} ${scale * 6} ${scale * 0.001}"/>
+      </geometry>
+      <origin xyz="0 0 ${scale * 0.009}"/>
+    </collision>
   </link>
   <joint name="base_with_middle_line" type="fixed">
@@ -95,4 +119,10 @@
       <material name="white"/>
     </visual>
+    <collision>
+      <geometry>
+        <box size="${scale * 9} ${scale * 6} ${scale * 0.001}"/>
+      </geometry>
+      <origin xyz="0 0 {scale * 0.001}"/>
+    </collision>
   </link>
   <joint name="base_with_outer_line" type="fixed">
@@ -109,4 +139,10 @@
       <material name="green"/>
     </visual>
+    <collision>
+     <geometry>
+        <box size="${scale * 8.84} ${scale * 5.84} ${scale * 0.001}"/>
+      </geometry>
+      <origin xyz="0 0 ${scale * 0.003}"/>
+    </collision>
   </link>
   <joint name="base_with_inner_field" type="fixed">
@@ -123,4 +159,10 @@
       <material name="white"/>
     </visual>
+    <collision>
+      <geometry>
+        <box size="${scale * 0.6} ${scale * 2.74} ${scale * 0.001}"/>
+      </geometry>
+      <origin xyz="${scale * -4.8} 0 ${scale * 0.001}"/>
+    </collision>
   </link>
   <joint name="base_with_goal_box_1" type="fixed">
@@ -137,4 +179,10 @@
       <material name="green"/>
     </visual>
+    <collision>
+      <geometry>
+        <box size="${scale * 0.52} ${scale * 2.6} ${scale * 0.001}"/>
+      </geometry>
+      <origin xyz="${scale * -4.76} 0 ${scale * 0.003}"/>
+    </collision>
   </link>
   <joint name="base_with_goal_area_1" type="fixed">
@@ -151,4 +199,10 @@
       <material name="white"/>
     </visual>
+    <collision>
+      <geometry>
+        <box size="${scale * 0.6} ${scale * 2.74} ${scale * 0.001}"/>
+      </geometry>
+      <origin xyz="${scale * 4.8} 0 ${scale * 0.001}"/>
+    </collision>
   </link>
   <joint name="base_with_goal_box_2" type="fixed">
@@ -165,4 +219,10 @@
       <material name="green"/>
     </visual>
+    <collision>
+      <geometry>
+        <box size="${scale * 0.52} ${scale * 2.6} ${scale * 0.001}"/>
+      </geometry>
+      <origin xyz="${scale * 4.76} 0 ${scale * 0.003}"/>
+    </collision>
   </link>
   <joint name="base_with_goal_area_2" type="fixed">
@@ -179,4 +239,10 @@
       <material name="white"/>
     </visual>
+    <collision>
+      <geometry>
+        <box size="${scale * 1} ${scale * 5} ${scale * 0.001}"/>
+      </geometry>
+      <origin xyz="${scale * -4} 0 ${scale * 0.005}"/>
+    </collision>
   </link>
   <joint name="base_with_penalty_box_1" type="fixed">
@@ -193,4 +259,10 @@
       <material name="green"/>
     </visual>
+    <collision>
+       <geometry>
+        <box size="${scale * 0.84} ${scale * 4.84} ${scale * 0.001}"/>
+      </geometry>
+      <origin xyz="${scale * -4} 0 ${scale * 0.007}"/>
+    </collision>
   </link>
   <joint name="base_with_penalty_area_1" type="fixed">
@@ -207,4 +279,10 @@
       <material name="white"/>
     </visual>
+    <collision>
+       <geometry>
+        <box size="${scale * 1} ${scale * 5} ${scale * 0.001}"/>
+      </geometry>
+      <origin xyz="${scale * 4} 0 ${scale * 0.005}"/>
+    </collision>
   </link>
   <joint name="base_with_penalty_box_2" type="fixed">
@@ -221,4 +299,10 @@
       <material name="green"/>
     </visual>
+    <collision>
+      <geometry>
+        <box size="${scale * 0.84} ${scale * 4.84} ${scale * 0.001}"/>
+      </geometry>
+      <origin xyz="${scale * 4} 0 ${scale * 0.007}"/>
+    </collision>
   </link>
   <joint name="base_with_penalty_area_2" type="fixed">
@@ -235,4 +319,10 @@
       <material name="white"/>
     </visual>
+    <collision>
+      <geometry>
+        <cylinder length ="${scale * 0.001}" radius="${scale * 0.075}"/>
+      </geometry>
+      <origin xyz="${scale  * -2.4} 0 ${scale * 0.005}"/>
+    </collision>
   </link>
   <joint name="base_with_penalty_mark_1" type="fixed">
@@ -249,4 +339,10 @@
       <material name="white"/>
     </visual>
+    <collision>
+      <geometry>
+        <cylinder length ="${scale * 0.001}" radius="${scale * 0.075}"/>
+      </geometry>
+      <origin xyz="${scale * 2.4} 0 ${scale * 0.005}"/>
+    </collision>
   </link>
   <joint name="base_with_penalty_mark_2" type="fixed">

File: urdf/robot.xacro (robot description, xacro)
@@ -2,4 +2,39 @@
 <robot name="UMARU" xmlns:xacro="http://www.ros.org/wiki/xacro">
   <xacro:property name="scale" value="1"/>
+  <xacro:property name="stack_length" value="0.04"/>
+  <xacro:property name="stack_width" value="0.04"/>
+  <xacro:property name="stack_tall" value="0.020"/>
+  <xacro:property name="stack_mass" value="0.98"/>
+  <xacro:macro name="empty_link" params="name">
+    <link name="${name}">
+      <inertial>
+        <mass value="0"/>
+        <inertia ixx="0" ixy="0" ixz="0" iyy="0" iyz="0" izz="0" />
+      </inertial>
+    </link>
+  </xacro:macro>
+  <xacro:macro name="stack_link" params="name">
+    <link name="${name}">
+      <visual>
+        <origin xyz="0 0 0"/>
+        <geometry>
+         <box size="${stack_length} ${stack_width} ${stack_tall}"/>
+       </geometry>
+      </visual>
+      <collision>
+        <origin xyz="0 0 0"/>
+       <geometry>
+          <box size="${stack_width} ${stack_width} ${stack_tall}"/>
+       </geometry>
+      </collision>
+      <inertial>
+       <mass value="stack_mass"/>
+       <origin xyz="0 0 0"/>
+       <inertia ixx="${stack_mass * (stack_width**2 + stack_tall**2) / 12}" ixy="0" ixz="0"
+               iyy="${stack_mass * (stack_width**2 + stack_tall**2) / 12}" iyz="0"
+               izz="${stack_mass * (stack_width**2 + stack_width**2) / 12}" />
+      </inertial>
+   </link>
+  </xacro:macro>
   <material name="cyan">
     <color rgba="0 255 255 1"/>
@@ -8,235 +43,626 @@
     <color rgba="255 255 0 1"/>
   </material>
-  <link name="world"></link>
+  <xacro:property name="body_length" value="0.117"/>
+  <xacro:property name="body_width" value="0.147"/>
+  <xacro:property name="body_tall" value="0.176124"/>
+  <xacro:property name="body_mass" value="1.80"/>
   <link name="body">
     <visual>
       <geometry>
-        <box size="${scale * 0.147}  ${scale * 0.117} ${scale * 0.176124}"/>
-      </geometry>
-      <origin rpy="0 0 1.57079632679"/>
+        <box size="${body_length}  ${body_width} ${body_tall}"/>
+      </geometry>
+      <origin rpy="0 0 0"/>
       <material name="cyan"/>
     </visual>
     <collision>
       <geometry>
-        <box size="${scale * 0.147}  ${scale * 0.117} ${scale * 0.176124}"/>
-      </geometry>
-      <origin rpy="0 0 1.57079632679"/>
-    </collision>
-  </link>
-  <joint name="body_with_world" type="fixed">
-    <parent link="world"/>
-    <child link="body"/>
-  </joint>
+        <box size="${body_length}  ${body_width} ${body_tall}"/>
+      </geometry>
+      <origin rpy="0 0 0"/>
+    </collision>
+    <inertial>
+      <mass value="${body_mass}"/>
+      <origin xyz="0 0 0"/>
+      <inertia ixx="${body_mass * (body_width**2 + body_tall**2) / 12}" ixy="0" ixz="0"
+               iyy="${body_mass * (body_length**2 + body_tall**2) / 12}" iyz="0"
+               izz="${body_mass * (body_width**2 + body_length**2) / 12}" />
+    </inertial>
+  </link>
+  <xacro:property name="h_sho_length" value="0.065"/>
+  <xacro:property name="h_sho_width" value="0.055"/>
+  <xacro:property name="h_sho_tall" value="0.030"/>
+  <xacro:property name="h_sho_mass" value="0.070"/>
   <link name="right_shoulder_horizontal">
     <visual>
       <geometry>
-        <box size="${scale * 0.055} ${scale * 0.065} ${scale * 0.030}"/>
-      </geometry>
-      <origin rpy="0 0 1.57079632679" xyz="0 0 0"/>
-      <material name="yellow"/>
-    </visual>
-    <collision>
-      <geometry>
-        <box size="${scale * 0.055} ${scale * 0.065} ${scale * 0.030}"/>
-      </geometry>
-      <origin rpy="0 0 1.57079632679" xyz="0 0 0"/>
-    </collision>
-  </link>
-  <joint name="R_SHO_PITCH" type="fixed"> <!-- JOINT_ID = 1 -->
-    <axis xyz="0 1 0"/>
+        <box size="${h_sho_length} ${h_sho_width} ${h_sho_tall}"/>
+      </geometry>
+      <origin rpy="0 0 0" xyz="0 ${- h_sho_width / 2} 0"/>
+      <material name="yellow"/>
+    </visual>
+    <collision>
+      <geometry>
+        <box size="${h_sho_length} ${h_sho_width} ${h_sho_tall}"/>
+      </geometry>
+      <origin rpy="0 0 0" xyz="0 ${- h_sho_width / 2} 0"/>
+    </collision>
+    <inertial>
+      <mass value="${h_sho_mass}"/>
+      <origin xyz="0 ${- h_sho_width / 2} 0"/>
+      <inertia ixx="${h_sho_mass * (h_sho_width**2 + h_sho_tall**2) / 12}" ixy="0" ixz="0"
+               iyy="${h_sho_mass * (h_sho_tall**2 + h_sho_length**2) / 12}" iyz="0"
+               izz="${h_sho_mass * (h_sho_width**2 + h_sho_length**2) / 12}" />
+    </inertial>
+  </link>
+  <link name="left_shoulder_horizontal">
+    <visual>
+      <geometry>
+         <box size="${h_sho_length} ${h_sho_width} ${h_sho_tall}"/>
+      </geometry>
+      <origin rpy="0 0 0" xyz="0 ${h_sho_width / 2} 0"/>
+      <material name="yellow"/>
+    </visual>
+    <collision>
+      <geometry>
+        <box size="${h_sho_length} ${h_sho_width} ${h_sho_tall}"/>
+      </geometry>
+      <origin rpy="0 0 0" xyz="0 ${h_sho_width / 2} 0"/>
+    </collision>
+    <inertial>
+      <mass value="${h_sho_mass}"/>
+      <origin xyz="0 ${h_sho_width / 2} 0"/>
+      <inertia ixx="${h_sho_mass * (h_sho_width**2 + h_sho_tall**2) / 12}" ixy="0" ixz="0"
+               iyy="${h_sho_mass * (h_sho_tall**2 + h_sho_length**2) / 12}" iyz="0"
+               izz="${h_sho_mass * (h_sho_width**2 + h_sho_length**2) / 12}" />
+    </inertial>
+  </link>
+  <xacro:property name="v_sho_length" value="0.065"/>
+  <xacro:property name="v_sho_width" value="0.030"/>
+  <xacro:property name="v_sho_tall" value="0.020"/>
+  <xacro:property name="v_sho_mass" value="0.070"/>
+  <link name="right_shoulder_vertical">
+    <visual>
+      <geometry>
+        <box size="${v_sho_length} ${v_sho_width} ${v_sho_tall}"/>
+      </geometry>
+      <origin rpy="0 0 0" xyz="0 0 ${- v_sho_tall / 2}"/>
+      <material name="yellow"/>
+    </visual>
+    <collision>
+      <geometry>
+        <box size="${v_sho_length} ${v_sho_width} ${v_sho_tall}"/>
+      </geometry>
+      <origin rpy="0 0 0" xyz="0 0 ${- v_sho_tall / 2}"/>
+    </collision>
+    <inertial>
+      <mass value="${v_sho_mass}"/>
+      <origin xyz="0 0 ${- v_sho_tall / 2}"/>
+      <inertia ixx="${v_sho_mass * (v_sho_width**2 + v_sho_tall**2) / 12}" ixy="0" ixz="0"
+               iyy="${v_sho_mass * (v_sho_length**2 + v_sho_tall**2) / 12}" iyz="0"
+               izz="${v_sho_mass * (v_sho_width**2 + v_sho_length**2) / 12}" />
+    </inertial>
+  </link>
+  <link name="left_shoulder_vertical">
+    <visual>
+      <geometry>
+        <box size="${v_sho_length} ${v_sho_width} ${v_sho_tall}"/>
+      </geometry>
+      <origin rpy="0 0 0" xyz="0 0 ${- v_sho_tall / 2}"/>
+      <material name="yellow"/>
+    </visual>
+    <collision>
+      <geometry>
+         <box size="${v_sho_length} ${v_sho_width} ${v_sho_tall}"/>
+      </geometry>
+      <origin rpy="0 0 0" xyz="0 0 ${- v_sho_tall / 2}"/>
+    </collision>
+    <inertial>
+      <mass value="${v_sho_mass}"/>
+      <origin xyz="0 0 ${- v_sho_tall / 2}"/>
+      <inertia ixx="${v_sho_mass * (v_sho_width**2 + v_sho_tall**2) / 12}" ixy="0" ixz="0"
+               iyy="${v_sho_mass * (v_sho_length**2 + v_sho_tall**2) / 12}" iyz="0"
+               izz="${v_sho_mass * (v_sho_width**2 + v_sho_length**2) / 12}" />
+    </inertial>
+  </link>
+  <xacro:property name="arm_length" value="0.038"/>
+  <xacro:property name="arm_width" value="0.0402"/>
+  <xacro:property name="arm_tall" value="0.156"/>
+  <xacro:property name="arm_mass" value="0.120"/>
+  <link name="right_arm">
+    <visual>
+      <geometry>
+        <box size="${arm_length} ${arm_width} ${arm_tall}"/>
+      </geometry>
+      <origin rpy="0 0 0" xyz="0 0 ${- arm_tall / 2}"/>
+      <material name="cyan"/>
+    </visual>
+    <collision>
+      <geometry>
+        <box size="${arm_length} ${arm_width} ${arm_tall}"/>
+      </geometry>
+      <origin rpy="0 0 0" xyz="0 0 ${- arm_tall / 2}"/>
+    </collision>
+    <inertial>
+      <mass value="${arm_mass}"/>
+      <origin xyz="0 0 ${- arm_tall / 2}"/>
+      <inertia ixx="${arm_mass * (arm_width**2 + arm_tall**2) / 12}" ixy="0" ixz="0"
+               iyy="${arm_mass * (arm_length**2 + arm_tall**2) / 12}" iyz="0"
+               izz="${arm_mass * (arm_width**2 + arm_length**2) / 12}" />
+    </inertial>
+  </link>
+  <link name="left_arm">
+    <visual>
+      <geometry>
+        <box size="${arm_length} ${arm_width} ${arm_tall}"/>
+      </geometry>
+      <origin rpy="0 0 0" xyz="0 0 ${- arm_tall / 2}"/>
+      <material name="cyan"/>
+    </visual>
+    <collision>
+      <geometry>
+        <box size="${arm_length} ${arm_width} ${arm_tall}"/>
+      </geometry>
+      <origin rpy="0 0 0" xyz="0 0 ${- arm_tall / 2}"/>
+    </collision>
+    <inertial>
+      <mass value="${arm_mass}"/>
+      <origin xyz="0 0 ${- arm_tall / 2}"/>
+      <inertia ixx="${arm_mass * (arm_width**2 + arm_tall**2) / 12}" ixy="0" ixz="0"
+               iyy="${arm_mass * (arm_length**2 + arm_tall**2) / 12}" iyz="0"
+               izz="${arm_mass * (arm_width**2 + arm_length**2) / 12}" />
+    </inertial>
+  </link>
+  <xacro:property name="hand_length" value="0.0276"/>
+  <xacro:property name="hand_width" value="0.0505"/>
+  <xacro:property name="hand_tall" value="0.162"/>
+  <xacro:property name="hand_mass" value="0.080"/>
+  <link name="right_hand">
+    <visual>
+      <geometry>
+        <box size="${hand_length} ${hand_width} ${hand_tall}"/>
+      </geometry>
+      <origin rpy="0 0 0" xyz="0 0 ${- hand_tall / 2}"/>
+      <material name="yellow"/>
+    </visual>
+    <collision>
+      <geometry>
+        <box size="${hand_length} ${hand_width} ${hand_tall}"/>
+      </geometry>
+      <origin rpy="0 0 0" xyz="0 0 ${- hand_tall / 2}"/>
+    </collision>
+    <inertial>
+      <mass value="${hand_mass}"/>
+      <origin xyz="0 0 ${- hand_tall / 2}"/>
+      <inertia ixx="${hand_mass * (hand_width**2 + hand_tall**2) / 12}" ixy="0" ixz="0"
+               iyy="${hand_mass * (hand_length**2 + hand_tall**2) / 12}" iyz="0"
+               izz="${hand_mass * (hand_width**2 + hand_length**2) / 12}" />
+    </inertial>
+  </link>
+  <link name="left_hand">
+    <visual>
+      <geometry>
+        <box size="${hand_length} ${hand_width} ${hand_tall}"/>
+      </geometry>
+      <origin rpy="0 0 0" xyz="0 0 ${- hand_tall / 2}"/>
+      <material name="yellow"/>
+    </visual>
+    <collision>
+      <geometry>
+        <box size="${hand_length} ${hand_width} ${hand_tall}"/>
+      </geometry>
+      <origin rpy="0 0 0" xyz="0 0 ${- hand_tall / 2}"/>
+    </collision>
+    <inertial>
+      <mass value="${hand_mass}"/>
+      <origin xyz="0 0 ${- hand_tall / 2}"/>
+      <inertia ixx="${hand_mass * (hand_width**2 + hand_tall**2) / 12}" ixy="0" ixz="0"
+               iyy="${hand_mass * (hand_length**2 + hand_tall**2) / 12}" iyz="0"
+               izz="${hand_mass * (hand_width**2 + hand_length**2) / 12}" />
+    </inertial>
+  </link>
+  <!-- EMPTY LINK-->
+  <xacro:empty_link name="head_tilt"/>
+  <xacro:empty_link name="right_hip"/>
+  <xacro:empty_link name="left_hip"/>
+  <xacro:property name="leg_width" value="0.049"/>
+  <xacro:property name="leg_tall" value="0.143"/>
+  <xacro:property name="leg_mass" value="0.300"/>
+<!-- HIP TEST WITH UPPER LEG EMPTY LINK -->
+  <!-- <xacro:property name="hip_tall" value="0.162"/>
+  <xacro:property name="hip_mass" value="0.120"/>
+  <link name="right_hip">
+    <visual>
+      <geometry>
+        <box size="${leg_width} ${leg_width} ${hip_tall}"/>
+      </geometry>
+      <origin xyz="0 0 ${- hip_tall/2}" rpy="0 0 0"/>
+      <material name="yellow"/>
+    </visual>
+    <collision>
+      <geometry>
+        <box size="${leg_width} ${leg_width} ${hip_tall}"/>
+      </geometry>
+      <origin xyz="0 0 ${- hip_tall/2}" rpy="0 0 0"/>
+    </collision>
+    <inertial>
+      <mass value="${hip_mass}"/>
+      <origin xyz="0 0 ${- hip_tall/2}"/>
+      <inertia ixx="${hip_mass * (leg_width**2 + hip_tall**2) / 12}" ixy="0" ixz="0"
+               iyy="${hip_mass * (leg_width**2 + hip_tall**2) / 12}" iyz="0"
+               izz="${hip_mass * (leg_width**2 + leg_width**2) / 12}" />
+    </inertial>
+  </link>
+  <link name="left_hip">
+    <visual>
+      <geometry>
+        <box size="${leg_width} ${leg_width} ${hip_tall}"/>
+      </geometry>
+      <origin rpy="0 0 0" xyz="0 0 ${- hip_tall/2}"/>
+      <material name="yellow"/>
+    </visual>
+    <collision>
+      <geometry>
+        <box size="${leg_width} ${leg_width} ${hip_tall}"/>
+      </geometry>
+      <origin rpy="0 0 0" xyz="0 0 ${- hip_tall/2}"/>
+    </collision>
+    <inertial>
+      <mass value="${hip_mass}"/>
+      <origin xyz="0 0 ${- hip_tall/2}"/>
+      <inertia ixx="${hip_mass * (leg_width**2 + hip_tall**2) / 12}" ixy="0" ixz="0"
+               iyy="${hip_mass * (leg_width**2 + hip_tall**2) / 12}" iyz="0"
+               izz="${hip_mass * (leg_width**2 + leg_width**2) / 12}" />
+    </inertial>
+  </link>  -->
+  <link name="left_upper_leg">
+    <visual>
+      <geometry>
+        <box size="${leg_width} ${leg_width} ${leg_tall}"/>
+      </geometry>
+      <origin xyz="0 0 ${- leg_tall/2}" rpy="0 0 0"/>
+      <material name="yellow"/>
+    </visual>
+    <collision>
+      <geometry>
+        <box size="${leg_width} ${leg_width} ${leg_tall}"/>
+      </geometry>
+      <origin xyz="0 0 ${- leg_tall/2}" rpy="0 0 0"/>
+    </collision>
+   <inertial>
+      <mass value="${leg_mass}"/>
+      <origin xyz="0 0 ${-leg_tall/2}"/>
+      <inertia ixx="${leg_mass* (leg_width**2 + leg_tall**2) / 12}" ixy="0" ixz="0"
+               iyy="${leg_mass * (leg_width**2 + leg_tall**2) / 12}" iyz="0"
+               izz="${leg_mass * (leg_width**2 + leg_width**2) / 12}" />
+    </inertial>
+  </link>
+  <link name="right_upper_leg">
+    <visual>
+      <geometry>
+        <box size="${leg_width} ${leg_width} ${leg_tall}"/>
+      </geometry>
+      <origin xyz="0 0 ${- leg_tall/2}" rpy="0 0  0"/>
+      <material name="yellow"/>
+    </visual>
+    <collision>
+      <geometry>
+        <box size="${leg_width} ${leg_width} ${leg_tall}"/>
+      </geometry>
+      <origin xyz="0 0 ${- leg_tall/2}" rpy="0 0 0"/>
+    </collision>
+     <inertial>
+      <mass value="${leg_mass}"/>
+      <origin xyz="0 0 ${-leg_tall/2}"/>
+      <inertia ixx="${leg_mass* (leg_width**2 + leg_tall**2) / 12}" ixy="0" ixz="0"
+               iyy="${leg_mass * (leg_width**2 + leg_tall**2) / 12}" iyz="0"
+               izz="${leg_mass * (leg_width**2 + leg_width**2) / 12}" />
+    </inertial>
+  </link>
+  <xacro:stack_link name="right_hip_roll"/>
+  <xacro:stack_link name="left_hip_roll"/>
+  <link name="left_lower_leg">
+    <visual>
+      <origin xyz="0 0 ${- leg_tall/2}" rpy="0 0 0" />
+      <material name="cyan" />
+      <geometry>
+        <box size="${leg_width} ${leg_width} ${leg_tall}" />
+      </geometry>
+    </visual>
+    <collision>
+      <origin xyz="0 0 ${- leg_tall/2}" rpy="0 0 0" />
+      <geometry>
+        <box size="${leg_width} ${leg_width} ${leg_tall}" />
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