Commit message: Removing unnecessary links and joints on the urdf file

File: urdf/robot.urdf (robot description, URDF)
Before this commit: robot UMARU, 24 links, 23 joints
Links:
- removed link head_tilt
Joints:
- removed joint NECK_TO_HEAD
- joint HEAD_TILT: origin xyz=0 0 0 -> xyz=0.0155 0 0; parent head_tilt -> neck
